File: YAWC_Cir/Micro.sch (KiCad schematic (older format))
At the start: 20 parts, among them P2 Btns, P3 CONN_5, P4 CONN_5, P5 CONN_6, U2 SAMD20J18A-M

Commit message: Add Keys project
Parts:
- C3, C4, C5, C6, C7: symbol C -> C-RESCUE-YAWC
- D1: symbol LED -> LED-RESCUE-YAWC
- R1, R4, R5: symbol R -> R-RESCUE-YAWC
Other:
- note added: "This is wrong. Need loop to +ve"
Changed lines of the file:
@@
 EESchema Schematic File Version 2
+LIBS:YAWC-rescue
 LIBS:power
 LIBS:device
@@
 LIBS:memory
 LIBS:xilinx
-LIBS:special
 LIBS:microcontrollers
 LIBS:dsp
@@
 LIBS:valves
 LIBS:YAWC-cache
-EELAYER 24 0
+EELAYER 25 0
 EELAYER END
 $Descr A4 11693 8268
@@
 VCC
 $Comp
-L C C3
+L C-RESCUE-YAWC C3
 U 1 1 53973676
 P 1150 1450
+AR Path="/53973676" Ref="C3"  Part="1"
+AR Path="/5394B774/53973676" Ref="C3"  Part="1"
 F 0 "C3" H 1150 1550 40  0000 L CNN
 F 1 "100n" H 1156 1365 40  0000 L CNN
@@
 $EndComp
 $Comp
-L C C4
+L C-RESCUE-YAWC C4
 U 1 1 539736A9
 P 1400 1450
+AR Path="/539736A9" Ref="C4"  Part="1"
+AR Path="/5394B774/539736A9" Ref="C4"  Part="1"
 F 0 "C4" H 1400 1550 40  0000 L CNN
 F 1 "100n" H 1406 1365 40  0000 L CNN
@@
 $EndComp
 $Comp
-L C C5
+L C-RESCUE-YAWC C5
 U 1 1 539736C2
 P 1650 1450
+AR Path="/539736C2" Ref="C5"  Part="1"
+AR Path="/5394B774/539736C2" Ref="C5"  Part="1"
 F 0 "C5" H 1650 1550 40  0000 L CNN
 F 1 "100n" H 1656 1365 40  0000 L CNN
@@
 $EndComp
 $Comp
-L C C6
+L C-RESCUE-YAWC C6
 U 1 1 539736DB
 P 1900 1450
+AR Path="/539736DB" Ref="C6"  Part="1"
+AR Path="/5394B774/539736DB" Ref="C6"  Part="1"
 F 0 "C6" H 1900 1550 40  0000 L CNN
 F 1 "100n" H 1906 1365 40  0000 L CNN
@@
 $EndComp
 $Comp
-L C C7
+L C-RESCUE-YAWC C7
 U 1 1 5397386B
 P 4550 1300
+AR Path="/5397386B" Ref="C7"  Part="1"
+AR Path="/5394B774/5397386B" Ref="C7"  Part="1"
 F 0 "C7" H 4550 1400 40  0000 L CNN
 F 1 "100n" H 4556 1215 40  0000 L CNN
@@
 $EndComp
 $Comp
-L GND #PWR04
+L GND-RESCUE-YAWC #PWR04
 U 1 1 539738BC
 P 4100 1400
@@
 VCC
 $Comp
-L R R1
+L R-RESCUE-YAWC R1
 U 1 1 53989FCC
 P 9700 1400
@@
 SWCLK
 $Comp
-L GND #PWR05
+L GND-RESCUE-YAWC #PWR05
 U 1 1 5398A8C9
 P 9700 2350
@@
 VCC
 $Comp
-L GND #PWR06
+L GND-RESCUE-YAWC #PWR06
 U 1 1 539AD64C
 P 10150 4150
@@
 $EndComp
 $Comp
-L R R4
+L R-RESCUE-YAWC R4
 U 1 1 539ADC21
 P 9700 4650
@@
 	7700 2750 7550 2750
 $Comp
-L LED D1
+L LED-RESCUE-YAWC D1
 U 1 1 539ED0A8
 P 3350 4050
@@
 	3550 4050 3850 4050
 $Comp
-L R R5
+L R-RESCUE-YAWC R5
 U 1 1 539ED159
 P 2750 4050
@@
 	950  2750 1150 2750
 $Comp
-L GND #PWR07
+L GND-RESCUE-YAWC #PWR07
 U 1 1 539EEC3B
 P 9950 3000
@@
 Connection ~ 950  2750
 $Comp
-L GND #PWR08
+L GND-RESCUE-YAWC #PWR08
 U 1 1 539EF45E
 P 5700 5400
@@
 Connection ~ 1750 1650
 $Comp
-L GND #PWR09
+L GND-RESCUE-YAWC #PWR09
 U 1 1 539EF936
 P 1500 1850
@@
 $EndComp
 $Comp
-L GND #PWR010
+L GND-RESCUE-YAWC #PWR010
 U 1 1 539EFA2D
 P 10000 5050
@@
 	9800 3350 9950 3350
 Connection ~ 9150 3650
+Text Notes 9100 5200 0    79   ~ 16
+This is wrong. Need loop to +ve
 $EndSCHEMATC
