File: YAWC_Breath/Breath_Amp.sch (KiCad schematic (older format))
At the start: 16 parts, among them P1 J_IO, P2 PressSens, U1 MCP6002, U2 MPX12DP

Commit message: Positioned connector and unrouted old
Parts:
- removed P2: PressSens, symbol CONN_2
- added BITE1: CONN_01X02, PIN_Hdr:Pin_Header_Angled_1x02, symbol CONN_01X02
- C1, C3, C4: footprint (none) -> Resistors_SMD:R_0805_HandSoldering; symbol C -> C-RESCUE-Breath_Amp
- C2: footprint (none) -> Capacitors_SMD:C_1206; symbol C -> C-RESCUE-Breath_Amp
- P1: footprint (none) -> PIN_Hdr:Pin_Header_Angled_1x04
- R1, R2, R3, R4, R5, R6, R7: footprint (none) -> Resistors_SMD:R_0805_HandSoldering; symbol R -> R-RESCUE-Breath_Amp
- RV1: footprint (none) -> VishTrim:TSM4YL
- U1: footprint (none) -> SMD_Packages:SOIC-8-N; symbol MCP6002 -> MCP6002-RESCUE-Breath_Amp
- U2: footprint (none) -> Sensors:MPX1351-01
Connections:
- wire segments 36 -> 42
Changed lines of the file:
@@
 EESchema Schematic File Version 2
+LIBS:Breath_Amp-rescue
 LIBS:power
 LIBS:device
@@
 LIBS:memory
 LIBS:xilinx
-LIBS:special
 LIBS:microcontrollers
 LIBS:dsp
@@
 LIBS:MyComponents
 LIBS:Breath_Amp-cache
-EELAYER 24 0
+EELAYER 25 0
 EELAYER END
 $Descr A4 11693 8268
@@
 $EndDescr
 $Comp
-L MCP6002 U1
+L MCP6002-RESCUE-Breath_Amp U1
 U 1 1 53920E78
 P 4000 2550
 F 0 "U1" H 4150 2700 60  0000 C CNN
 F 1 "MCP6002" H 4200 2350 60  0000 C CNN
-F 2 "" H 4000 2550 60  0000 C CNN
+F 2 "SMD_Packages:SOIC-8-N" H 4000 2550 60  0001 C CNN
 F 3 "" H 4000 2550 60  0000 C CNN
 F 4 "133-2118" H 4000 2550 60  0001 C CNN "F#"
@@
 $EndComp
 $Comp
-L MCP6002 U1
+L MCP6002-RESCUE-Breath_Amp U1
 U 2 1 53920EC1
 P 6650 2550
 F 0 "U1" H 6800 2700 60  0000 C CNN
 F 1 "MCP6002" H 6850 2350 60  0000 C CNN
-F 2 "" H 6650 2550 60  0000 C CNN
+F 2 "SMD_Packages:SOIC-8-N" H 6650 2550 60  0001 C CNN
 F 3 "" H 6650 2550 60  0000 C CNN
 	2    6650 2550
@@
 $EndComp
 $Comp
-L GND #PWR01
+L GND-RESCUE-Breath_Amp #PWR01
 U 1 1 53920FC5
 P 3900 2950
@@
 $EndComp
 $Comp
-L GND #PWR02
+L GND-RESCUE-Breath_Amp #PWR02
 U 1 1 53920FE1
 P 6550 3200
@@
 Wire Wire Line
 	6550 3200 6550 2950
-Text GLabel 3900 1400 1    60   Input ~ 0
-VCC
 Text Label 3900 2150 0    60   ~ 0
 VCC
@@
 F 0 "P1" V 8900 1500 50  0000 C CNN
 F 1 "J_IO" V 9000 1500 50  0000 C CNN
-F 2 "" H 8950 1500 60  0000 C CNN
+F 2 "PIN_Hdr:Pin_Header_Angled_1x04" H 8950 1500 60  0001 C CNN
 F 3 "" H 8950 1500 60  0000 C CNN
 	1    8950 1500
@@
 Pout
 $Comp
-L C C2
+L C-RESCUE-Breath_Amp C2
 U 1 1 53921326
 P 7650 1350
 F 0 "C2" H 7650 1450 40  0000 L CNN
 F 1 "1u" H 7656 1265 40  0000 L CNN
-F 2 "" H 7688 1200 30  0000 C CNN
+F 2 "Capacitors_SMD:C_1206" H 7688 1200 30  0001 C CNN
 F 3 "" H 7650 1350 60  0000 C CNN
 	1    7650 1350
@@
 $EndComp
 $Comp
-L GND #PWR03
+L GND-RESCUE-Breath_Amp #PWR03
 U 1 1 53921361
 P 7650 1550
@@
 F 0 "RV1" H 3150 1800 50  0000 C CNN
 F 1 "100k" H 3150 1900 50  0000 C CNN
-F 2 "" H 3150 1900 60  0000 C CNN
+F 2 "VishTrim:TSM4YL" H 3150 1900 60  0001 C CNN
 F 3 "" H 3150 1900 60  0000 C CNN
 F 4 "114-1366" H 3150 1900 60  0001 C CNN "F#"
@@
 $EndComp
 Wire Wire Line
-	3900 1400 3150 1400
+	3150 1400 6550 1400
 Wire Wire Line
 	3150 1400 3150 1650
@@
 F 0 "U2" H 1650 2500 60  0000 C CNN
 F 1 "MPX12DP" H 1650 2250 60  0000 C CNN
-F 2 "" H 1650 2500 60  0000 C CNN
+F 2 "Sensors:MPX1351-01" H 1650 2500 60  0001 C CNN
 F 3 "" H 1650 2500 60  0000 C CNN
 	1    1650 2500
@@
 $EndComp
 $Comp
-L GND #PWR04
+L GND-RESCUE-Breath_Amp #PWR04
 U 1 1 5392CBCA
 P 2100 2900
@@
 	1450 2650 2100 2650
 $Comp
-L R R2
+L R-RESCUE-Breath_Amp R2
 U 1 1 5392CBFD
 P 2650 2550
 F 0 "R2" V 2730 2550 40  0000 C CNN
 F 1 "10k" V 2657 2551 40  0000 C CNN
-F 2 "" V 2580 2550 30  0000 C CNN
+F 2 "Resistors_SMD:R_0805_HandSoldering" V 2580 2550 30  0001 C CNN
 F 3 "" H 2650 2550 30  0000 C CNN
 	1    2650 2550
@@
 $EndComp
 $Comp
-L R R3
+L R-RESCUE-Breath_Amp R3
 U 1 1 5392CC46
 P 2950 3000
 F 0 "R3" V 3030 3000 40  0000 C CNN
 F 1 "150k" V 2957 3001 40  0000 C CNN
-F 2 "" V 2880 3000 30  0000 C CNN
+F 2 "Resistors_SMD:R_0805_HandSoldering" V 2880 3000 30  0001 C CNN
 F 3 "" H 2950 3000 30  0000 C CNN
 	1    2950 3000
@@
 $EndComp
 $Comp
-L R R4
+L R-RESCUE-Breath_Amp R4
 U 1 1 5392CC65
 P 3900 3250
 F 0 "R4" V 3980 3250 40  0000 C CNN
 F 1 "150k" V 3907 3251 40  0000 C CNN
-F 2 "" V 3830 3250 30  0000 C CNN
+F 2 "Resistors_SMD:R_0805_HandSoldering" V 3830 3250 30  0001 C CNN
 F 3 "" H 3900 3250 30  0000 C CNN
 	1    3900 3250
@@
 $EndComp
 $Comp
-L R R1
+L R-RESCUE-Breath_Amp R1
 U 1 1 5392CC96
 P 2650 2350
 F 0 "R1" V 2730 2350 40  0000 C CNN
 F 1 "10k" V 2657 2351 40  0000 C CNN
-F 2 "" V 2580 2350 30  0000 C CNN
+F 2 "Resistors_SMD:R_0805_HandSoldering" V 2580 2350 30  0001 C CNN
 F 3 "" H 2650 2350 30  0000 C CNN
 	1    2650 2350
@@
 Connection ~ 2950 2550
 $Comp
-L GND #PWR05
+L GND-RESCUE-Breath_Amp #PWR05
 U 1 1 5392CD6C
 P 2950 3350
@@
 	4500 2450 4500 3500
 $Comp
-L C C1
+L C-RESCUE-Breath_Amp C1
 U 1 1 5392CEB2
 P 3900 3500
 F 0 "C1" H 3900 3600 40  0000 L CNN
 F 1 "2n" H 3906 3415 40  0000 L CNN
-F 2 "" H 3938 3350 30  0000 C CNN
+F 2 "Resistors_SMD:R_0805_HandSoldering" H 3938 3350 30  0001 C CNN
 F 3 "" H 3900 3500 60  0000 C CNN
 	1    3900 3500
@@
 VCC
 $Comp
-L R R6
+L R-RESCUE-Breath_Amp R6
 U 1 1 5392E54F
 P 5750 2450
 F 0 "R6" V 5830 2450 40  0000 C CNN
 F 1 "3600" V 5757 2451 40  0000 C CNN
-F 2 "" V 5680 2450 30  0000 C CNN
+F 2 "Resistors_SMD:R_0805_HandSoldering" V 5680 2450 30  0001 C CNN
 F 3 "" H 5750 2450 30  0000 C CNN
 	1    5750 2450
@@
 $EndComp
 $Comp
-L R R5
+L R-RESCUE-Breath_Amp R5
 U 1 1 5392E5E2
 P 5050 2450
 F 0 "R5" V 5130 2450 40  0000 C CNN
 F 1 "316" V 5057 2451 40  0000 C CNN
-F 2 "" V 4980 2450 30  0000 C CNN
+F 2 "Resistors_SMD:R_0805_HandSoldering" V 4980 2450 30  0001 C CNN
 F 3 "" H 5050 2450 30  0000 C CNN
 	1    5050 2450
@@
 	6000 2450 6150 2450
 $Comp
-L C C4
+L C-RESCUE-Breath_Amp C4
 U 1 1 5392E68F
 P 6000 2750
 F 0 "C4" H 6000 2850 40  0000 L CNN
 F 1 "82n" H 6006 2665 40  0000 L CNN
-F 2 "" H 6038 2600 30  0000 C CNN
+F 2 "Resistors_SMD:R_0805_HandSoldering" H 6038 2600 30  0001 C CNN
 F 3 "" H 6000 2750 60  0000 C CNN
 	1    6000 2750
@@
 $EndComp
 $Comp
-L C C3
+L C-RESCUE-Breath_Amp C3
 U 1 1 5392E6C2
 P 5750 1950
 F 0 "C3" H 5750 2050 40  0000 L CNN
 F 1 "820n" H 5756 1865 40  0000 L CNN
-F 2 "" H 5788 1800 30  0000 C CNN
+F 2 "Resistors_SMD:R_0805_HandSoldering" H 5788 1800 30  0001 C CNN
 F 3 "" H 5750 1950 60  0000 C CNN
 	1    5750 1950
@@
 VCC
 $Comp
-L CONN_2 P2
-U 1 1 5393315D
-P 1550 4300
-F 0 "P2" V 1500 4300 40  0000 C CNN
-F 1 "PressSens" V 1600 4300 40  0000 C CNN
-F 2 "" H 1550 4300 60  0000 C CNN
-F 3 "" H 1550 4300 60  0000 C CNN
-	1    1550 4300
-	-1   0    0    -1
-$EndComp
-$Comp
-L R R7
+L R-RESCUE-Breath_Amp R7
 U 1 1 539331B2
 P 2000 3800
 F 0 "R7" V 2080 3800 40  0000 C CNN
 F 1 "100" V 2007 3801 40  0000 C CNN
-F 2 "" V 1930 3800 30  0000 C CNN
+F 2 "Resistors_SMD:R_0805_HandSoldering" V 1930 3800 30  0001 C CNN
 F 3 "" H 2000 3800 30  0000 C CNN
 	1    2000 3800
@@
 $EndComp
 Wire Wire Line
-	1900 4200 2600 4200
+	1650 4200 2600 4200
 Wire Wire Line
 	2000 4200 2000 4050
 Wire Wire Line
-	1900 4400 2150 4400
+	1650 4400 2150 4400
 Wire Wire Line
 	2150 4400 2150 4450
 $Comp
-L GND #PWR06
+L GND-RESCUE-Breath_Amp #PWR06
 U 1 1 539332B6
 P 2150 4450
@@
 Text Label 2600 4200 0    60   ~ 0
 Pout
+Wire Wire Line
+	3150 2150 3150 3250
+Wire Wire Line
+	3150 3250 2950 3250
+$Comp
+L CONN_01X02 BITE1
+U 1 1 5708EF62
+P 1450 4300
+F 0 "BITE1" H 1450 4450 50  0000 C CNN
+F 1 "CONN_01X02" V 1550 4300 50  0000 C CNN
+F 2 "PIN_Hdr:Pin_Header_Angled_1x02" H 1450 4300 50  0001 C CNN
+F 3 "" H 1450 4300 50  0000 C CNN
+	1    1450 4300
+	-1   0    0    1
+$EndComp
+Wire Wire Line
+	1650 4250 1650 4200
+Wire Wire Line
+	1650 4400 1650 4350
+Connection ~ 3900 1400
+Wire Wire Line
+	3900 2150 3900 1400
+Wire Wire Line
+	6550 1400 6550 2150
 $EndSCHEMATC
